Commit message: correcting the height of 3dsensor

File: waiterbot_suite/waiterbot_bringup/urdf/waiterbot_v2.urdf (robot description, URDF)
Before this commit: robot turtlebot, 27 links, 26 joints
Joints:
- joint camera_rgb_joint: origin xyz=-0.0389 0.0205 0.325 rpy=0 0 0 -> xyz=-0.0389 0.0205 0.355 rpy=0 0 0
